File: aqua_control_rcv/aqua_control_rcv.kicad_sch (KiCad schematic)
At the start: 51 parts, among them J1 USB_C, J4 Conn_01x03, J5 Conn_01x03, Q1 MMBT2222A, Q2 IRLML6402, SW1 RESET, SW2 BOOT, SW3 BOOT, SW4 BOOT, U1 ESP32-S3-WROOM-1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

Commit message: routing completed
Parts:
- removed J2, J3: (no value), TerminalBlock:TerminalBlock_MaiXu_MX126-5.0-03P_1x03_P5.00mm, symbol Connector:Screw_Terminal_01x03
- added J2, J3: Screw_Terminal_01x04, TerminalBlock:TerminalBlock_MaiXu_MX126-5.0-04P_1x04_P5.00mm, symbol Connector:Screw_Terminal_01x04
Connections:
- net 3.3v: now also R16.2; no longer R16.1
- net Earth: now also J2.4 (Pin_4), J3.4 (Pin_4)
- net L_in: now also J2.1 (Pin_1), J2.2 (Pin_2)
- net L_out: now also J3.1 (Pin_1), J3.2 (Pin_2)
- net N_in: now also J2.3 (Pin_3), J3.3 (Pin_3)
- net at C2.1, C3.1, U2.2 (VO): now also R16.1; no longer R16.2
Other:
- moved on the sheet: R16

Commit message: receiver board complete
Parts:
- D1: footprint Diode_THT:D_DO-41_SOD81_P10.16mm_Horizontal -> Diode_SMD:D_SMA
- SW1, SW2, SW3, SW4: footprint Button_Switch_THT:SW_DIP_SPSTx01_Slide_6.7x4.1mm_W7.62mm_P2.54mm_LowProfile -> sw_smd:SW_TS09-63-25-WT-160-SMT-TR
Changed lines of the file:
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@@
 			)
 		)
-		(property "Footprint" "Button_Switch_THT:SW_DIP_SPSTx01_Slide_6.7x4.1mm_W7.62mm_P2.54mm_LowProfile"
+		(property "Footprint" "sw_smd:SW_TS09-63-25-WT-160-SMT-TR"
 			(at 52.07 123.19 0)
 			(hide yes)
@@
 			)
 		)
-		(property "Footprint" "Button_Switch_THT:SW_DIP_SPSTx01_Slide_6.7x4.1mm_W7.62mm_P2.54mm_LowProfile"
+		(property "Footprint" "sw_smd:SW_TS09-63-25-WT-160-SMT-TR"
 			(at 168.91 172.72 0)
 			(hide yes)
@@
 			)
 		)
-		(property "Footprint" "Diode_THT:D_DO-41_SOD81_P10.16mm_Horizontal"
+		(property "Footprint" "Diode_SMD:D_SMA"
 			(at 87.63 182.245 0)
 			(hide yes)
@@
 			)
 		)
-		(property "Footprint" "Button_Switch_THT:SW_DIP_SPSTx01_Slide_6.7x4.1mm_W7.62mm_P2.54mm_LowProfile"
+		(property "Footprint" "sw_smd:SW_TS09-63-25-WT-160-SMT-TR"
 			(at 142.24 172.72 0)
 			(hide yes)
@@
 			)
 		)
-		(property "Footprint" "Button_Switch_THT:SW_DIP_SPSTx01_Slide_6.7x4.1mm_W7.62mm_P2.54mm_LowProfile"
+		(property "Footprint" "sw_smd:SW_TS09-63-25-WT-160-SMT-TR"
 			(at 85.09 121.92 0)
 			(hide yes)
